File: P00F.kicad_pcb (KiCad board)
At the start: 2 copper layers, 37.7 x 48.1 mm, 6 parts, among them J1 UJ20-C-H-G-SMT-TR, J2 TYPE-C-31-M-12, J3 USB4120-03-C_REVA

Commit message: Update Bom and PCB_top
Other:
- board text added: "Type-C_compilation ID:P00F <<version>> 2024-11-11 Git-36f7bdb www.website.com//P00F"
- board text removed: "<<project_name>> <<ID>> <<version>> <<date>> <<hash>> <<website_link>>"
Changed lines of the file:
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@@
 	(paper "A4")
 	(title_block
-		(title "<<ID>>_<<project_name>>")
-		(date "<<date>>")
+		(title "ID:P00F_Type-C_compilation")
+		(date "2024-11-11")
 		(rev "<<version>>")
-		(comment 4 "<<hash>>")
+		(comment 4 "Git-36f7bdb")
 	)
 	(layers
@@
 		(layer "Edge.Cuts")
 	)
-	(gr_text "<<project_name>>\n<<ID>>\n<<version>>\n<<date>>\n<<hash>>\n<<website_link>>"
+	(gr_text "Type-C_compilation\nID:P00F\n<<version>>\n2024-11-11\nGit-36f7bdb\nwww.website.com//P00F"
 		(at 225.75 151 0)
 		(layer "F.SilkS")
