File: P00F.kicad_sch (KiCad schematic)
At the start: 6 parts, among them J1 UJ20-C-H-G-SMT-TR, J2 TYPE-C-31-M-12, J3 USB4120-03-C_REVA

Commit message: Update Bom and PCB_top
Other:
- title: <<ID>>_<<project_name>> -> P00F_Type-C_compilation
Changed lines of the file:
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@@
 	(paper "A4")
 	(title_block
-		(title "<<ID>>_<<project_name>>")
-		(date "<<date>>")
+		(title "P00F_Type-C_compilation")
+		(date "2024-11-04")
 		(rev "<<version>>")
-		(comment 4 "<<hash>>")
+		(comment 4 "Git-079f43a")
 	)
 	(symbol
