File: P00F.kicad_sch (KiCad schematic)
At the start: 6 parts, among them J1 UJ20-C-H-G-SMT-TR, J2 TYPE-C-31-M-12, J3 USB4120-03-C_REVA

Commit message: fake change
Other:
- moved on the sheet: J1
Changed lines of the file:
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@@
 	(symbol
 		(lib_id "Snapeda_kicad_sym:UJ20-C-H-G-SMT-TR")
-		(at 120.65 58.42 0)
+		(at 113.03 59.69 0)
 		(unit 1)
 		(exclude_from_sim no)
@@
 		(fields_autoplaced yes)
 		(property "Reference" "J1"
-			(at 120.65 30.48 0)
+			(at 113.03 31.75 0)
 			(effects
 				(font
@@
 		)
 		(property "Value" "UJ20-C-H-G-SMT-TR"
-			(at 120.65 33.02 0)
+			(at 113.03 34.29 0)
 			(effects
 				(font
@@
 		)
 		(property "Footprint" "Snapeda:UJ20-C-H-G-SMT-TR_CUI_UJ20-C-H-G-SMT-TR"
-			(at 120.65 58.42 0)
+			(at 113.03 59.69 0)
 			(effects
 				(font
@@
 		)
 		(property "Datasheet" ""
-			(at 120.65 58.42 0)
+			(at 113.03 59.69 0)
 			(effects
 				(font
@@
 		)
 		(property "Description" ""
-			(at 120.65 58.42 0)
+			(at 113.03 59.69 0)
 			(effects
 				(font
@@
 		)
 		(property "MF" "CUI Devices"
-			(at 120.65 58.42 0)
+			(at 113.03 59.69 0)
 			(effects
 				(font
@@
 		)
 		(property "MAXIMUM_PACKAGE_HEIGHT" "3.66mm"
-			(at 120.65 58.42 0)
+			(at 113.03 59.69 0)
 			(effects
 				(font
@@
 		)
 		(property "Package" "None"
-			(at 120.65 58.42 0)
+			(at 113.03 59.69 0)
 			(effects
 				(font
@@
 		)
 		(property "Price" "None"
-			(at 120.65 58.42 0)
+			(at 113.03 59.69 0)
 			(effects
 				(font
@@
 		)
 		(property "Check_prices" "https://www.snapeda.com/parts/UJ20-C-H-G-SMT-TR/Same+Sky/view-part/?ref=eda"
-			(at 120.65 58.42 0)
+			(at 113.03 59.69 0)
 			(effects
 				(font
@@
 		)
 		(property "STANDARD" "Manufacturer Recommendations"
-			(at 120.65 58.42 0)
+			(at 113.03 59.69 0)
 			(effects
 				(font
@@
 		)
 		(property "PARTREV" "1.01"
-			(at 120.65 58.42 0)
+			(at 113.03 59.69 0)
 			(effects
 				(font
@@
 		)
 		(property "SnapEDA_Link" "https://www.snapeda.com/parts/UJ20-C-H-G-SMT-TR/Same+Sky/view-part/?ref=snap"
-			(at 120.65 58.42 0)
+			(at 113.03 59.69 0)
 			(effects
 				(font
@@
 		)
 		(property "MP" "UJ20-C-H-G-SMT-TR"
-			(at 120.65 58.42 0)
+			(at 113.03 59.69 0)
 			(effects
 				(font
@@
 		)
 		(property "Purchase-URL" "https://www.snapeda.com/api/url_track_click_mouser/?unipart_id=12123263&manufacturer=CUI Devices&part_name=UJ20-C-H-G-SMT-TR&search_term=uj20-c-h-g-smt-tr"
-			(at 120.65 58.42 0)
+			(at 113.03 59.69 0)
 			(effects
 				(font
@@
 		)
 		(property "Description_1" "Type C, USB 2.0, 480 Mbps, 20 Vdc, 5 A, Right Angle, Gold Flash, Surface Mount, Black Insulator, USB Receptacle"
-			(at 120.65 58.42 0)
+			(at 113.03 59.69 0)
 			(effects
 				(font
@@
 		)
 		(property "CUI_purchase_URL" "https://www.cuidevices.com/product/interconnect/connectors/usb-connectors/uj20-c-h-g-smt-tr?utm_source=snapeda.com&utm_medium=referral&utm_campaign=snapedaBOM"
-			(at 120.65 58.42 0)
+			(at 113.03 59.69 0)
 			(effects
 				(font
@@
 		)
 		(property "Availability" "In Stock"
-			(at 120.65 58.42 0)
+			(at 113.03 59.69 0)
 			(effects
 				(font
@@
 		)
 		(property "MANUFACTURER" "CUI Devices"
-			(at 120.65 58.42 0)
+			(at 113.03 59.69 0)
 			(effects
 				(font

Commit message: Update Bom and PCB_top
Other:
- title: <<ID>>_<<project_name>> -> P00F_Type-C_compilation
Changed lines of the file:
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@@
 	(paper "A4")
 	(title_block
-		(title "<<ID>>_<<project_name>>")
-		(date "<<date>>")
+		(title "P00F_Type-C_compilation")
+		(date "2024-11-11")
 		(rev "<<version>>")
-		(comment 4 "<<hash>>")
+		(comment 4 "Git-36f7bdb")
 	)
 	(symbol
